Commit message: add fast_livo, camera_sim

File: src/ttbot_description/urdf/ttbot.urdf.xacro (robot description, xacro)
@@ -249,4 +249,34 @@
     <origin xyz="0.1 0 ${wheel_radius + chassis_height + 0.13}" rpy="0 0 0"/>
     <axis xyz="0 0 0"/>
+  </joint>
+  <!-- ================= CAMERA LINK ================= -->
+  <link name="camera_link">
+    <visual>
+      <geometry>
+        <box size="0.025 0.09 0.025"/>
+      </geometry>
+      <material name="blue"><color rgba="0 0 1 1"/></material>
+    </visual>
+    <collision>
+      <geometry>
+        <box size="0.025 0.09 0.025"/>
+      </geometry>
+    </collision>
+    <inertial>
+      <mass value="0.05"/>
+      <origin xyz="0 0 0" rpy="0 0 0"/>
+      <inertia ixx="1e-6" ixy="0" ixz="0" iyy="1e-6" iyz="0" izz="1e-6"/>
+    </inertial>
+  </link>
+  <joint name="camera_joint" type="fixed">
+    <parent link="base_link"/>
+    <child link="camera_link"/>
+    <origin xyz="0.5 0 ${wheel_radius + chassis_height + 0.05}" rpy="0 0 0"/>
+  </joint>
+  <link name="camera_color_optical_frame"></link>
+  <joint name="camera_optical_joint" type="fixed">
+    <parent link="camera_link"/>
+    <child link="camera_color_optical_frame"/>
+    <origin xyz="0 0 0" rpy="-1.57079632679 0 -1.57079632679"/>
   </joint>
   <!-- ================= ROS2_CONTROL ================= -->

File: src/ttbot_description/urdf/ttbot_gazebo.xacro (robot description, xacro)
@@ -57,5 +57,5 @@
     <sensor name="imu" type="imu">
         <always_on>true</always_on>
-        <update_rate>100</update_rate>
+        <update_rate>400</update_rate>
         <gz_frame_id>imu_link</gz_frame_id>
         <topic>imu</topic>
@@ -149,4 +149,46 @@
       </sensor>
   </gazebo>
+  <gazebo reference="camera_link">
+    <sensor name="realsense_d435i_rgbd" type="rgbd_camera">
+      <pose>0 0 0 0 0 0</pose>
+      <always_on>true</always_on>
+      <update_rate>30</update_rate>
+      <topic>/camera/rgbd</topic>
+      <ignition_frame_id>camera_color_optical_frame</ignition_frame_id>
+      <camera>
+        <horizontal_fov>1.5184</horizontal_fov>
+        <image>
+          <width>640</width>
+          <height>480</height>
+          <format>R8G8B8</format>
+        </image>
+        <clip>
+          <near>0.1</near>
+          <far>10.0</far> </clip>
+      </camera>
+    </sensor>
+    <sensor name="realsense_d435i_imu" type="imu">
+      <always_on>true</always_on>
+      <update_rate>200</update_rate> <topic>/camera/imu</topic>
+      <ignition_frame_id>camera_link</ignition_frame_id>
+      <imu>
+        <angular_velocity>
+          <x><noise type="gaussian"><mean>0.0</mean><stddev>2e-4</stddev></noise></x>
+          <y><noise type="gaussian"><mean>0.0</mean><stddev>2e-4</stddev></noise></y>
+          <z><noise type="gaussian"><mean>0.0</mean><stddev>2e-4</stddev></noise></z>
+        </angular_velocity>
+        <linear_acceleration>
+          <x><noise type="gaussian"><mean>0.0</mean><stddev>1.7e-2</stddev></noise></x>
+          <y><noise type="gaussian"><mean>0.0</mean><stddev>1.7e-2</stddev></noise></y>
+          <z><noise type="gaussian"><mean>0.0</mean><stddev>1.7e-2</stddev></noise></z>
+        </linear_acceleration>
+      </imu>
+    </sensor>
+  </gazebo>
+  <!-- <gazebo>
+    <plugin filename="ignition-gazebo-sensors-system" name="ignition::gazebo::systems::Sensors">
+      <render_engine>ogre2</render_engine>
+    </plugin>
+  </gazebo> -->
   <gazebo>
       <plugin filename="ignition-gazebo-navsat-system"

Commit message: update

File: src/ttbot_description/urdf/ttbot.urdf.xacro (robot description, xacro)
@@ -209,5 +209,5 @@
     <parent link="base_link"/>
     <child link="lidar_link"/>
-    <origin xyz="0 0 ${wheel_radius + chassis_height + 0.2}" rpy="0 0 0"/>
+    <origin xyz="-0.30 -0.03 1.50" rpy="0 0 0"/>
   </joint>
   <!-- ================= IMU JOINT ================= -->
@@ -215,6 +215,5 @@
     <parent link="base_link"/>
     <child link="imu_link"/>
-    <origin xyz="0 0 ${wheel_radius + chassis_height + 0.13}" rpy="0 0 0"/>
-    <axis xyz="0 0 0"/>
+    <origin xyz="-0.20 -0.03 1.50" rpy="0 0 0"/>
   </joint>
   <!-- ================= GPS LINK ================= -->
@@ -272,5 +271,5 @@
     <parent link="base_link"/>
     <child link="camera_link"/>
-    <origin xyz="0.5 0 ${wheel_radius + chassis_height + 0.05}" rpy="0 0 0"/>
+    <origin xyz="-0.20 -0.05 1.46" rpy="0 0 0"/>
   </joint>
   <link name="camera_color_optical_frame"></link>

Commit message: remove grid in gazebo

File: src/ttbot_description/urdf/ttbot.urdf.xacro (robot description, xacro)
@@ -117,5 +117,4 @@
   <xacro:wheel_link name="rear_left_wheel"/>
   <xacro:wheel_link name="rear_right_wheel"/>
-  <!-- ================= JOINTS ================= -->
   <joint name="front_left_steering_joint" type="revolute">
     <parent link="base_link"/>
@@ -157,5 +156,112 @@
     <axis xyz="0 1 0"/>
   </joint>
-  <!-- ================= IMU LINK ================= -->
+  <link name="sensor_tower_link">
+    <visual>
+      <origin xyz="0 0.15 0.53" rpy="0 0 0"/>
+      <geometry><box size="0.04 0.04 1.06"/></geometry>
+      <material name="gray"><color rgba="0.5 0.5 0.5 1"/></material>
+    </visual>
+    <collision>
+      <origin xyz="0 0.15 0.53" rpy="0 0 0"/>
+      <geometry><box size="0.04 0.04 1.06"/></geometry>
+    </collision>
+    <visual>
+      <origin xyz="0 -0.15 0.53" rpy="0 0 0"/>
+      <geometry><box size="0.04 0.04 1.06"/></geometry>
+      <material name="gray"><color rgba="0.5 0.5 0.5 1"/></material>
+    </visual>
+    <collision>
+      <origin xyz="0 -0.15 0.53" rpy="0 0 0"/>
+      <geometry><box size="0.04 0.04 1.06"/></geometry>
+    </collision>
+    <visual>
+      <origin xyz="0 0 1.04" rpy="0 0 0"/>
+      <geometry><box size="0.04 0.34 0.04"/></geometry>
+      <material name="gray"><color rgba="0.5 0.5 0.5 1"/></material>
+    </visual>
+    <collision>
+      <origin xyz="0 0 1.04" rpy="0 0 0"/>
+      <geometry><box size="0.04 0.34 0.04"/></geometry>
+    </collision>
+    <visual>
+      <origin xyz="0 0 0.5" rpy="0 0 0"/>
+      <geometry><box size="0.04 0.45 0.04"/></geometry>
+      <material name="gray"><color rgba="0.5 0.5 0.5 1"/></material>
+    </visual>
+    <collision>
+      <origin xyz="0 0 0.5" rpy="0 0 0"/>
+      <geometry><box size="0.04 0.45 0.04"/></geometry>
+    </collision>
+    <inertial>
+      <mass value="1.5"/>
+      <origin xyz="0 0 0.53" rpy="0 0 0"/>
+      <inertia ixx="0.14" ixy="0" ixz="0" iyy="0.14" iyz="0" izz="0.02"/>
+    </inertial>
+  </link>
+  <joint name="sensor_tower_joint" type="fixed">
+    <parent link="base_link"/>
+    <child link="sensor_tower_link"/>
+    <origin xyz="-0.2 0 ${wheel_radius + chassis_height}" rpy="0 0 0"/>
+  </joint>
+  <link name="laptop_tray_link">
+    <visual>
+      <origin xyz="-0.18 0.15 0" rpy="0 0 0"/>
+      <geometry><box size="0.36 0.04 0.04"/></geometry>
+      <material name="gray"><color rgba="0.5 0.5 0.5 1"/></material>
+    </visual>
+    <collision>
+      <origin xyz="-0.18 0.15 0" rpy="0 0 0"/>
+      <geometry><box size="0.36 0.04 0.04"/></geometry>
+    </collision>
+    <visual>
+      <origin xyz="-0.18 -0.15 0" rpy="0 0 0"/>
+      <geometry><box size="0.36 0.04 0.04"/></geometry>
+      <material name="gray"><color rgba="0.5 0.5 0.5 1"/></material>
+    </visual>
+    <collision>
+      <origin xyz="-0.18 -0.15 0" rpy="0 0 0"/>
+      <geometry><box size="0.36 0.04 0.04"/></geometry>
+    </collision>
+    <visual>
+      <origin xyz="-0.18 0 0.025" rpy="0 0 0"/>
+      <geometry><box size="0.28 0.34 0.01"/></geometry>
+      <material name="black"><color rgba="0.1 0.1 0.1 1"/></material>
+    </visual>
+    <collision>
+      <origin xyz="-0.18 0 0.025" rpy="0 0 0"/>
+      <geometry><box size="0.28 0.34 0.01"/></geometry>
+    </collision>
+    <inertial>
+      <mass value="1.0"/>
+      <origin xyz="-0.18 0 0" rpy="0 0 0"/>
+      <inertia ixx="0.01" ixy="0" ixz="0" iyy="0.01" iyz="0" izz="0.01"/>
+    </inertial>
+  </link>
+  <joint name="laptop_tray_joint" type="fixed">
+    <parent link="sensor_tower_link"/>
+    <child link="laptop_tray_link"/>
+    <origin xyz="-0.02 0 0.15" rpy="0 0 0"/>
+  </joint>
+  <link name="sensor_box_link">
+    <visual>
+      <origin xyz="0 0 0" rpy="0 0 0"/>
+      <geometry><box size="0.2 0.25 0.1"/></geometry>
+      <material name="white"><color rgba="0.9 0.9 0.9 1"/></material>
+    </visual>
+    <collision>
+      <origin xyz="0 0 0" rpy="0 0 0"/>
+      <geometry><box size="0.2 0.25 0.1"/></geometry>
+    </collision>
+    <inertial>
+      <mass value="0.5"/>
+      <origin xyz="0 0 0" rpy="0 0 0"/>
+      <inertia ixx="0.003" ixy="0" ixz="0" iyy="0.002" iyz="0" izz="0.004"/>
+    </inertial>
+  </link>
+  <joint name="sensor_box_joint" type="fixed">
+    <parent link="sensor_tower_link"/>
+    <child link="sensor_box_link"/>
+    <origin xyz="0 0 1.1" rpy="0 0 0"/>
+  </joint>
   <link name="imu_link">
     <visual>
@@ -182,5 +288,4 @@
     </inertial>
   </link>
-  <!-- ================= LIDAR LINK ================= -->
   <link name="lidar_link">
     <visual>
@@ -205,17 +310,14 @@
     </inertial>
   </link>
-  <!-- ================= LIDAR JOINT ================= -->
   <joint name="lidar_joint" type="fixed">
-    <parent link="base_link"/>
+    <parent link="sensor_box_link"/>
     <child link="lidar_link"/>
-    <origin xyz="-0.30 -0.03 1.50" rpy="0 0 0"/>
-  </joint>
-  <!-- ================= IMU JOINT ================= -->
+    <origin xyz="0 0 0.085" rpy="0 0 0"/>
+  </joint>
   <joint name="imu_joint" type="fixed">
-    <parent link="base_link"/>
+    <parent link="sensor_box_link"/>
     <child link="imu_link"/>
-    <origin xyz="-0.20 -0.03 1.50" rpy="0 0 0"/>
-  </joint>
-  <!-- ================= GPS LINK ================= -->
+    <origin xyz="0 0 0" rpy="0 0 0"/>
+  </joint>
   <link name="gps_link">
     <visual>
@@ -242,5 +344,4 @@
     </inertial>
   </link>
-  <!-- ================= GPS JOINT ================= -->
   <joint name="gps_joint" type="fixed">
     <parent link="base_link"/>
@@ -249,5 +350,4 @@
     <axis xyz="0 0 0"/>
   </joint>
-  <!-- ================= CAMERA LINK ================= -->
   <link name="camera_link">
     <visual>
@@ -269,7 +369,7 @@
   </link>
   <joint name="camera_joint" type="fixed">
-    <parent link="base_link"/>
+    <parent link="sensor_box_link"/>
     <child link="camera_link"/>
-    <origin xyz="-0.20 -0.05 1.46" rpy="0 0 0"/>
+    <origin xyz="0.1 0 0" rpy="0 0 0"/>
   </joint>
   <link name="camera_color_optical_frame"></link>
@@ -279,5 +379,4 @@
     <origin xyz="0 0 0" rpy="-1.57079632679 0 -1.57079632679"/>
   </joint>
-  <!-- ================= ROS2_CONTROL ================= -->
   <ros2_control name="ttbot_system" type="system">
     <hardware>
@@ -288,4 +387,6 @@
         <plugin>gz_ros2_control/GazeboSystem</plugin>
       </xacro:unless>
+      <param name="passive_joint">front_left_wheel_joint</param>
+      <param name="passive_joint">front_right_wheel_joint</param>
     </hardware>
     <joint name="rear_left_wheel_joint">
